Commit message: move group interface

File: robot/urdf/robot.urdf (robot description, URDF)
Before this commit: robot robot, 9 links, 8 joints
Joints:
- joint joint1: origin xyz=0 0 0.06 rpy=1.5708 0 0.21073 -> xyz=0 0 0.06 rpy=1.5708 0 0
- joint joint7: origin xyz=-0.049867 -0.079042 0 rpy=0 0.61703 -3.1416 -> xyz=-0.049867 -0.079042 0 rpy=0 0 0
